File: PCB/Rheneium.kicad_pcb (KiCad board)
At the start: 2 copper layers, 357.2 x 134.9 mm, 210 parts, among them J1 Conn_01x04_Pin, SW1 ESC, SW10 SW_Push, SW11 SW_Push, SW12 SW_Push, SW13 SW_Push, SW14 SW_Push, SW15 SW_Push, SW16 SW_Push, SW17 SW_Push, SW18 SW_Push, SW19 SW_Push, SW2 SW_Push, SW20 SW_Push, SW21 SW_Push, SW22 SW_Push, SW23 SW_Push, SW24 SW_Push, SW25 SW_Push, SW26 SW_Push, SW27 SW_Push, SW28 SW_Push, SW29 SW_Push, SW3 SW_Push, SW30 SW_Push, SW31 SW_Push, SW32 SW_Push, SW33 SW_Push, SW34 SW_Push, SW35 SW_Push, SW36 SW_Push, SW37 SW_Push, SW38 SW_Push, SW39 SW_Push, SW4 SW_Push, SW40 SW_Push, SW41 SW_Push, SW42 SW_Push, SW43 SW_Push, SW44 SW_Push, SW45 SW_Push, SW46 SW_Push, SW47 SW_Push, SW48 SW_Push, SW49 SW_Push, SW5 SW_Push, SW50 SW_Push, SW51 SW_Push, SW52 SW_PUSH, SW53 SW_Push, SW54 SW_Push, SW55 SW_Push, SW56 SW_Push, SW57 SW_Push, SW58 SW_Push, SW59 SW_Push, SW6 SW_Push, SW60 SW_Push, SW61 SW_Push, SW62 SW_Push, SW63 SW_Push, SW64 SW_Push, SW65 SW_Push, SW66 SW_Push, SW67 SW_Push, SW68 SW_Push, SW69 SW_Push, SW7 SW_Push, SW70 SW_Push, SW71 SW_Push, SW74 SW_Push, SW75 SW_Push, SW76 SW_Push, SW77 SW_Push, SW78 SW_Push, SW79 SW_Push, SW8 SW_Push, SW80 SW_Push, SW81 SW_Push, SW82 SW_Push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

Commit message: Add files via upload
Parts:
- C15, C6, C7, C8, R9: moved to B.Cu
- C9, D84, X1: moved to F.Cu
- moved C8 28.8 mm to (308.0, 101.6)
- moved C15 24.9 mm to (313.5, 101.9), turned to 90 degrees
- moved R1 24.2 mm to (317.5, 111.1), turned to 180 degrees
- moved C4 22.4 mm to (308.0, 103.2), turned to 180 degrees
- moved C2 18.4 mm to (308.8, 107.5)
- moved C6 17.8 mm to (315.9, 109.1)
- moved C7 16.8 mm to (318.3, 103.5)
- moved C5 14.4 mm to (317.8, 109.0), turned to 0 degrees
- moved X1 14.1 mm to (298.9, 103.1), turned to 0 degrees
- moved C3 10.4 mm to (318.6, 106.9), turned to 0 degrees
- moved C1 7.53 mm to (318.3, 108.0), turned to 0 degrees
- moved C12 7.17 mm to (325.4, 109.4)
- moved C9 6.04 mm to (302.7, 103.2)
- moved U4 5.25 mm to (321.8, 109.4)
- moved JP2 4.14 mm to (341.5, 106.4), turned to 180 degrees
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Routing:
- net GND: track 196.9 -> 338.2 mm
- net COL_3: track 518.4 -> 463.8 mm
- net COL_5: track 623.3 -> 571.7 mm
- net COL_6: track 532.5 -> 484.6 mm
- net COL_7: track 349.4 -> 304.4 mm
- net COL_8: track 327.8 -> 284.7 mm
- net COL_4: track 492.3 -> 454.3 mm
- net COL_9: track 494.0 -> 456.4 mm
- net COL_10: track 414.5 -> 378.1 mm
- net COL_11: track 331.9 -> 297.1 mm
- net COL_13: track 293.0 -> 258.9 mm
- net COL_12: track 273.1 -> 239.2 mm
- net COL_1: track 596.5 -> 572.7 mm
- net 23: track 33.2 -> 54.2 mm
- net ROW_6: track 395.0 -> 374.1 mm, vias 7 -> 10
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Other:
- board size 357.2 x 134.9 mm -> 358.8 x 134.9 mm

Commit message: Add files via upload
Parts:
- removed R7: 1K, Resistor_SMD:R_0402_1005Metric
- C10, C15, C6, C7, C8, R9: moved to F.Cu
- moved C10 14.3 mm to (299.2, 105.6), turned to 0 degrees
- moved C8 11.1 mm to (318.8, 104.3), turned to 0 degrees
- moved C6 6.53 mm to (318.8, 103.2), turned to 0 degrees
- moved C15 5.37 mm to (318.8, 100.8), turned to 180 degrees
- moved C7 1.53 mm to (318.7, 102.0), turned to 0 degrees
- moved R9 1.02 mm to (308.5, 104.8)
Routing:
- net Net-(C10-Pad1): track 21.4 -> 1.97 mm, vias 1 -> 0
- net XOUT: track 11.1 -> 0.00 mm, vias 3 -> 0
- net COL_4: track 454.3 -> 459.4 mm, vias 2 -> 4
- net RS_2: track 38.6 -> 43.4 mm, vias 0 -> 2
- net COL_2: track 452.4 -> 456.1 mm, vias 0 -> 2
- net RS_1: track 31.6 -> 35.3 mm, vias 0 -> 2
- net COL_1: track 572.7 -> 576.4 mm, vias 0 -> 2
- net COL_3: track 463.8 -> 467.2 mm, vias 1 -> 3
- net 3V3: track 176.8 -> 174.2 mm, vias 9 -> 5
- net GND: track 338.2 -> 336.5 mm, vias 8 -> 9
- net gp2: track 75.1 -> 76.6 mm
- net ROW_2: track 367.5 -> 368.8 mm
- net 23: track 54.2 -> 55.3 mm
- net 25: track 2.25 -> 1.18 mm, vias 1 -> 0
- net USB_DM_CLEAN: track 27.0 -> 26.0 mm
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
Commit message: Add files via upload
Routing:
- net 3V3: track 174.2 -> 303.4 mm, vias 5 -> 16
- net ROW_6: track 374.1 -> 405.3 mm, vias 10 -> 11
- net 1V1: track 4.84 -> 17.4 mm, vias 0 -> 4
- net GND: track 336.5 -> 343.4 mm, vias 9 -> 11
Other:
- board text added: "Built By Shreyansh aka Endinvoid"

Commit message: Add files via upload
Routing:
- net 3V3: track 303.4 -> 304.8 mm, vias 16 -> 15
Changed lines of the file:
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@@
-	)
-	(segment
-		(start 341.3125 112.7125)
-		(end 330.99375 112.7125)
-		(width 0.2)
-		(layer "F.Cu")
-		(net 105)
 	)
 	(segment
@@
 	)
 	(segment
-		(start 330.71 91.28125)
-		(end 344.4875 91.28125)
-		(width 0.2)
-		(layer "F.Cu")
-		(net 105)
-	)
-	(segment
-		(start 308.76875 107.95)
-		(end 309.5625 107.15625)
-		(width 0.2)
-		(layer "F.Cu")
-		(net 105)
-	)
-	(segment
 		(start 318.29375 110.84125)
 		(end 318.29375 109.78225)
@@
 	)
 	(segment
-		(start 312.893765 109.606265)
-		(end 313.61875 110.33125)
-		(width 0.2)
-		(layer "F.Cu")
-		(net 105)
-	)
-	(segment
 		(start 338.611251 103.98125)
 		(end 338.93125 103.98125)
@@
 	)
 	(segment
-		(start 348.45625 95.25)
-		(end 348.45625 105.56875)
-		(width 0.2)
-		(layer "F.Cu")
-		(net 105)
-	)
-	(segment
-		(start 309.5625 107.15625)
-		(end 309.578171 107.15625)
-		(width 0.2)
-		(layer "F.Cu")
-		(net 105)
-	)
-	(segment
 		(start 318.26375 102.04375)
 		(end 318.26375 103.1575)
@@
 	)
 	(segment
+		(start 346.86875 91.28125)
+		(end 330.71 91.28125)
+		(width 0.2)
+		(layer "F.Cu")
+		(net 105)
+	)
+	(segment
 		(start 320.675 108.43125)
 		(end 321.876 107.23025)
@@
 	)
 	(segment
-		(start 309.578171 107.15625)
-		(end 309.578585 107.156664)
+		(start 348.45625 106.3625)
+		(end 348.45625 92.86875)
 		(width 0.2)
 		(layer "F.Cu")
@@
 	)
 	(segment
-		(start 344.4875 91.28125)
-		(end 348.45625 95.25)
-		(width 0.2)
-		(layer "F.Cu")
-		(net 105)
-	)
-	(segment
 		(start 310.09375 106.58125)
 		(end 310.93125 107.41875)
@@
 	)
 	(segment
-		(start 348.45625 105.56875)
-		(end 341.3125 112.7125)
-		(width 0.2)
-		(layer "F.Cu")
-		(net 105)
-	)
-	(segment
 		(start 318.84735 109.78225)
 		(end 319.486675 109.142925)
@@
 	)
 	(segment
-		(start 309.5625 107.15625)
+		(start 308.76875 107.95)
 		(end 310.09375 106.625)
 		(width 0.2)
@@
 	)
 	(segment
+		(start 340.51875 114.3)
+		(end 348.45625 106.3625)
+		(width 0.2)
+		(layer "F.Cu")
+		(net 105)
+	)
+	(segment
 		(start 313.61875 110.33125)
 		(end 312.753804 110.33125)
@@
 	)
 	(segment
+		(start 329.40625 114.3)
+		(end 340.51875 114.3)
+		(width 0.2)
+		(layer "F.Cu")
+		(net 105)
+	)
+	(segment
 		(start 312.753804 110.33125)
 		(end 312.753599 110.331455)
@@
 	)
 	(segment
+		(start 348.45625 92.86875)
+		(end 346.86875 91.28125)
+		(width 0.2)
+		(layer "F.Cu")
+		(net 105)
+	)
+	(segment
 		(start 336.011251 106.58125)
 		(end 337.9775 104.615)
@@
 	)
 	(segment
-		(start 312.93125 107.41875)
-		(end 312.93125 109.074567)
-		(width 0.2)
-		(layer "F.Cu")
-		(net 105)
-	)
-	(segment
 		(start 318.0875 102.98125)
 		(end 318.29375 103.1875)
@@
 	)
 	(via
+		(at 317.5 88.9)
+		(size 0.6)
+		(drill 0.3)
+		(layers "F.Cu" "B.Cu")
+		(net 105)
+	)
+	(via
+		(at 338.93125 46.83125)
+		(size 0.6)
+		(drill 0.3)
+		(layers "F.Cu" "B.Cu")
+		(net 105)
+	)
+	(via
 		(at 329.40625 114.3)
-		(size 0.6)
-		(drill 0.3)
-		(layers "F.Cu" "B.Cu")
-		(net 105)
-	)
-	(via
-		(at 317.5 88.9)
-		(size 0.6)
-		(drill 0.3)
-		(layers "F.Cu" "B.Cu")
-		(net 105)
-	)
-	(via
-		(at 338.93125 46.83125)
 		(size 0.6)
 		(drill 0.3)
@@
 	)
 	(via
-		(at 309.578585 107.156664)
-		(size 0.6)
-		(drill 0.3)
-		(layers "F.Cu" "B.Cu")
-		(net 105)
-	)
-	(via
 		(at 306.3875 102.39375)
 		(size 0.6)
@@
 	(segment
 		(start 329.40625 114.3)
-		(end 330.99375 112.7125)
+		(end 337.9775 105.72875)
 		(width 0.2)
 		(layer "B.Cu")
@@
 	)
 	(segment
-		(start 330.99375 112.7125)
-		(end 337.9775 105.72875)
-		(width 0.2)
-		(layer "B.Cu")
-		(net 105)
-	)
-	(segment
 		(start 313.846921 99.21875)
 		(end 313.346263 99.719408)
@@
 	)
 	(segment
-		(start 308.83125 102.39375)
-		(end 308.76875 102.33125)
-		(width 0.2)
-		(layer "B.Cu")
-		(net 107)
-	)
-	(segment
 		(start 297.8375 104.6425)
 		(end 298.76375 105.56875)
@@
 		(start 309.8125 108.8275)
 		(end 309.5625 108.5775)
-		(width 0.2)
-		(layer "F.Cu")
-		(net 109)
-	)
-	(segment
-		(start 312.93125 100.54375)
-		(end 312.93125 100.999)
 		(width 0.2)
 		(layer "F.Cu")
@@
 	)
 	(segment
-		(start 312.752144 101.585356)
-		(end 312.7375 101.6)
-		(width 0.2)
-		(layer "B.Cu")
-		(net 109)
-	)
-	(segment
 		(start 313.53125 102.39375)
 		(end 313.53125 106.3625)
@@
 		(width 0.2)
 		(layer "F.Cu")
-		(net 124)
-	)
-	(segment
-		(start 314.61875 109.0375)
-		(end 314.61875 108.971351)
-		(width 0.2)
-		(layer "F.Cu")

Commit message: Add files via upload
Parts:
- moved C2 0.34 mm to (308.4, 107.5), turned to -135 degrees
- moved C13 0.31 mm to (309.6, 108.7)
- moved R9 0.14 mm to (308.4, 104.7)
Routing:
- net ROW_2: track 368.9 -> 367.4 mm
- net Net-(D88-A): track 3.18 -> 3.91 mm
- net 3V3: track 304.8 -> 305.4 mm
- net 25: track 1.18 -> 1.77 mm
